File: kicad/output-cape-v1.kicad_pcb (KiCad board)
At the start: 2 copper layers, 60.4 x 86.4 mm, 121 parts, among them J101 Conn_01x16_Female, J102 Conn_01x16_Female, J103 24V, Q1001 2N7002, Q1101 2N7002, Q1201 2N7002, Q1301 2N7002, Q1401 2N7002, Q1501 2N7002, Q1601 2N7002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

Commit message: add final V1 production files
Parts:
- JP102, JP103: footprint Connector_PinHeader_1.27mm:PinHeader_2x01_P1.27mm_Vertical_SMD -> Jumper:SolderJumper-2_P1.3mm_Open_TrianglePad1.0x1.5mm
- moved JP102 2.70 mm to (105.0, 116.2)
- moved JP103 2.70 mm to (107.5, 116.2)
- moved REF** 0.45 mm to (96.0, 139.5)
- moved REF** 0.45 mm to (103.0, 139.5)
- moved REF** 0.45 mm to (110.0, 139.5)
- moved REF** 0.45 mm to (117.0, 139.5), turned to 180 degrees
- moved R108 0.20 mm to (109.3, 115.5)
- moved R107 0.15 mm to (103.2, 115.5)
Routing:
- net /SW1_A1: track 7.37 -> 4.39 mm
- net /SW1_A2: track 7.07 -> 4.40 mm
- net +3V3: track 83.0 -> 84.0 mm
- net GNDD: track 80.7 -> 81.6 mm, vias 54 -> 196
Other:
- board text removed: "A1"
- board text removed: "A2"
