File: kicad/output-cape-v1.sch (KiCad schematic (older format))
At the start: 37 parts, among them J101 Conn_01x16_Female, J102 Conn_01x16_Female, J103 24V, U101 LM317_TO-252, U102 AT24C256C-SSHL-T, U103 BBB_P9, U104 BBB_P8

Commit message: add final V1 production files
Parts:
- JP102, JP103: footprint Connector_PinHeader_1.27mm:PinHeader_2x01_P1.27mm_Vertical_SMD -> Jumper:SolderJumper-2_P1.3mm_Open_TrianglePad1.0x1.5mm; symbol Device:Jumper_NO_Small -> Jumper:SolderJumper_2_Open
Changed lines of the file:
@@
 $EndComp
 $Comp
-L Device:Jumper_NO_Small JP103
+L Jumper:SolderJumper_2_Open JP103
 U 1 1 60C83D17
 P 8250 6050
 F 0 "JP103" H 8250 5957 50  0000 C CNN
 F 1 "A2" H 8250 5866 50  0000 C CNN
-F 2 "Connector_PinHeader_1.27mm:PinHeader_2x01_P1.27mm_Vertical_SMD" H 8250 6050 50  0001 C CNN
+F 2 "Jumper:SolderJumper-2_P1.3mm_Open_TrianglePad1.0x1.5mm" H 8250 6050 50  0001 C CNN
 F 3 "~" H 8250 6050 50  0001 C CNN
 F 4 "0" H 8250 6050 50  0001 C CNN "JLCPCB BOM"
@@
 $EndComp
 $Comp
-L Device:Jumper_NO_Small JP102
+L Jumper:SolderJumper_2_Open JP102
 U 1 1 60C84177
 P 8250 5950
 F 0 "JP102" H 8250 6135 50  0000 C CNN
 F 1 "A1" H 8250 6044 50  0000 C CNN
-F 2 "Connector_PinHeader_1.27mm:PinHeader_2x01_P1.27mm_Vertical_SMD" H 8250 5950 50  0001 C CNN
+F 2 "Jumper:SolderJumper-2_P1.3mm_Open_TrianglePad1.0x1.5mm" H 8250 5950 50  0001 C CNN
 F 3 "~" H 8250 5950 50  0001 C CNN
 F 4 "0" H 8250 5950 50  0001 C CNN "JLCPCB BOM"
@@
 	8850 5950 8850 5900
 Wire Wire Line
-	8700 6050 8350 6050
+	8700 6050 8400 6050
 Connection ~ 8700 6050
-Wire Wire Line
-	8850 5950 8350 5950
-Connection ~ 8850 5950
 $Comp
 L Device:R_Small R108
@@
 	8050 6100 8050 6050
 Wire Wire Line
-	8050 6050 8150 6050
-Wire Wire Line
-	8150 5950 8050 5950
+	8050 6050 8100 6050
 Wire Wire Line
 	8050 5950 8050 6050
@@
 	0    -1   -1   0
 $EndComp
+Wire Wire Line
+	8850 5950 8400 5950
+Connection ~ 8850 5950
+Wire Wire Line
+	8100 5950 8050 5950
 $EndSCHEMATC
